File: Electronics/EMHarpsichord_Sustainer+Playback/EMHarpsichord_Sustainer+Playback.kicad_pcb (KiCad board)
At the start: 2 copper layers, 61.2 x 27.4 mm, 50 parts, among them J1 Conn_01x03_Male, J2 Conn_01x04_Male, J3 Conn_01x03_Male, U1 ITR20403, U2 NE5532, U3 PAM8406D

Commit message: More tidying files and adding comments to schematics
Other:
- board text added: "Electromagnetic Harpsichord Project: Optical Sustainer V1 (Sep 21, 2023)"
- board text removed: "Electromagnetic Harpsichord Project: Optical Sustainer"
- board text removed: "This optical sustainer board connects the terminals of speaker ouptuts on an audio power amplifier chip (PAM8406) to the ends of a metal (often brass) string. When a signal is input to the board, a correlated current moves back and forth on the string and consequently an alternating magnetic field is generated along the string. When that string is in the presence of a strong magnetic field (perha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"
- board text removed: "max length: 40mm"
- board text removed: "max width: 10mm"
Changed lines of the file:
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@@
     (effects (font (size 1 1) (thickness 0.15)))
   )
-  (gr_text "This optical sustainer board connects the terminals of speaker ouptuts on an audio power amplifier chip (PAM8406)\nto the ends of a metal (often brass) string. When a signal is input to the board, a correlated current \nmoves back and forth on the string and consequently an alternating magnetic field is generated along the string.\nWhen that string is in the presence of a strong magnetic field (perhaps a strong neodynium magnet), the string's \nmagnetic field interacts with the neodynium magnet's, inducing mechancial vibration into the string.\n\nAn optical sensor (ITR20403) is used to 'pickup' a signal analogous to the position of the string.\nA differentiator circuit takes the deriviative of this signal to create a signal analagous to the\nvelocity of the string. When this signal is fed into the power amplifier connected to the strings,\na feedback loop is created and the natural vibrations on the string are sustained.\n\nThe left channel is an optical sensor to sustain a string connected to its outputs.\nThe right channel takes an auxillary input signal and puts that signal on a different string." (at 124.968 140.081) (layer "Cmts.User")
+  (gr_text "Electromagnetic Harpsichord Project: Optical Sustainer V1 (Sep 21, 2023)" (at 125.476 91.44) (layer "Cmts.User")
     (effects (font (size 1 1) (thickness 0.15)) (justify left))
   )
-  (gr_text "Electromagnetic Harpsichord Project: Optical Sustainer" (at 125.476 91.44) (layer "Cmts.User")
+  (gr_text "Left Channel is for sustain\nRight Channel is for audio playback" (at 125.603 86.868) (layer "Cmts.User")
     (effects (font (size 1 1) (thickness 0.15)) (justify left))
   )
-  (gr_text "max length: 40mm\n" (at 133.35 78.232) (layer "Cmts.User")
-    (effects (font (size 1 1) (thickness 0.15)))
-  )
-  (gr_text "Left Channel is for sustain\nRight Channel is for audio playback" (at 125.95 81.294) (layer "Cmts.User")
-    (effects (font (size 1 1) (thickness 0.15)) (justify left))
-  )
-  (gr_text "max width: 10mm\n" (at 133.062 76.214) (layer "Cmts.User")
-    (effects (font (size 1 1) (thickness 0.15)))
-  )
   (segment (start 152.146 97.155) (end 156.6585 97.155) (width 0.4) (layer "F.Cu") (net 1))
